File: hardware/roadster-charger/boost.kicad_sch (KiCad schematic)
At the start: 29 parts, among them U10 DAC70501ZDQFT, U11 PI3740-00-LGIZ

Commit message: one more big grounding change
Parts:
- added TP12: TestPoint_Alt, TestPoint:TestPoint_THTPad_D1.0mm_Drill0.5mm, symbol Connector:TestPoint_Alt
Connections:
- net PGND is gone; now on net GND: C18.2, C19.2, C20.2, C21.2, C22.2, C26.2, C27.2, C28.2, C29.2, C30.2, C31.2, C32.2, C33.2, U11.B2 (PGND), U11.B3 (PGND), U11.B4 (PGND), U11.B5 (PGND), U11.B6 (PGND), U11.B7 (PGND), U11.B8 (PGND), U11.B9 (PGND), U11.C2 (PGND), U11.C3 (PGND), U11.C4 (PGND), U11.C5 (PGND), U11.C6 (PGND), U11.C7 (PGND), U11.C8 (PGND), U11.C9 (PGND), U11.D2 (PGND), U11.D3 (PGND), U11.D4 (PGND), U11.D5 (PGND), U11.D6 (PGND), U11.D7 (PGND), U11.D8 (PGND), U11.D9 (PGND), U11.E2 (PGND), U11.E3 (PGND), U11.E4 (PGND), U11.E5 (PGND), U11.E6 (PGND), U11.E7 (PGND), U11.E8 (PGND), U11.E9 (PGND), U11.F7 (PGND), U11.F8 (PGND), U11.G7 (PGND), U11.G8 (PGND), U11.H7 (PGND), U11.H8 (PGND), U11.J7 (PGND), U11.J8 (PGND), U11.K7 (PGND), U11.K8 (PGND)
- net GND: now also TP12.1; no longer C17.2, C23.2, C24.2, C25.2, R26.2, U10.3 (AGND), U10.6 (*SYNC/A0), U11.A1 (FT1), U11.A10 (VSP), U11.A2 (FT2), U11.A3 (FT3), U11.A4 (FT4), U11.A7 (LGH), U11.B1 (SYNCI), U11.B10 (SGND), U11.B11 (SGND), U11.B12 (SGND), U11.B13 (SGND), U11.B14 (SGND), U11.C10 (SGND), U11.C11 (SGND), U11.C12 (SGND), U11.D10 (SGND), U11.D11 (SGND), U11.D12 (SGND), U11.D14 (ISN), U11.E10 (SGND), U11.E11 (SGND), U11.E12 (SGND), U11.E14 (ISP)
- new net SGND: C17.2, C23.2, C24.2, C25.2, R26.2, U10.3 (AGND), U10.6 (*SYNC/A0), U11.A1 (FT1), U11.A10 (VSP), U11.A2 (FT2), U11.A3 (FT3), U11.A4 (FT4), U11.A7 (LGH), U11.B1 (SYNCI), U11.B10 (SGND), U11.B11 (SGND), U11.B12 (SGND), U11.B13 (SGND), U11.B14 (SGND), U11.C10 (SGND), U11.C11 (SGND), U11.C12 (SGND), U11.D10 (SGND), U11.D11 (SGND), U11.D12 (SGND), U11.D14 (ISN), U11.E10 (SGND), U11.E11 (SGND), U11.E12 (SGND), U11.E14 (ISP)
Other:
- note added: "This testpoint in case some GND reference reworks need to be done to the DAC"

Commit message: Fix res PN, remove TPs from BOM, add DNPs to BOM
Parts:
- JP1: MPN (none) -> DNP
- TP10, TP11, TP8, TP9: now left out of the parts list
- TP12: MPN (none) -> DNP; now left out of the parts list
Changed lines of the file:
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@@
 		(unit 1)
 		(exclude_from_sim no)
-		(in_bom yes)
+		(in_bom no)
 		(on_board yes)
 		(dnp no)
@@
 		(unit 1)
 		(exclude_from_sim no)
-		(in_bom yes)
+		(in_bom no)
 		(on_board yes)
 		(dnp no)
@@
 			)
 		)
+		(property "MPN" "DNP"
+			(at 115.57 152.4 0)
+			(effects
+				(font
+					(size 1.27 1.27)
+				)
+				(hide yes)
+			)
+		)
 		(pin "1"
 		)
@@
 		(unit 1)
 		(exclude_from_sim no)
-		(in_bom yes)
+		(in_bom no)
 		(on_board yes)
 		(dnp no)
@@
 		(unit 1)
 		(exclude_from_sim no)
-		(in_bom yes)
+		(in_bom no)
 		(on_board yes)
 		(dnp no)
@@
 		(unit 1)
 		(exclude_from_sim no)
-		(in_bom yes)
+		(in_bom no)
 		(on_board yes)
 		(dnp no)
@@
 			(at 175.26 138.43 0)
 			(effects
+				(font
+					(size 1.27 1.27)
+				)
+				(hide yes)
+			)
+		)
+		(property "MPN" "DNP"
+			(at 175.26 138.43 0)
+			(effects

Commit message: Undo DNPs in BOM, update cap PN
Parts:
- C18, C19, C20, C21, C22, C26, C27, C28, C29, C30, C31, C32, C33: MPN GRM32ER72A225KA35 -> GRM32ER72A225KA35L
Changed lines of the file:
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@@
 			)
 		)
-		(property "MPN" "GRM32ER72A225KA35"
+		(property "MPN" "GRM32ER72A225KA35L"
 			(at 151.13 107.95 0)
 			(effects
@@
 			)
 		)
-		(property "MPN" "GRM32ER72A225KA35"
+		(property "MPN" "GRM32ER72A225KA35L"
 			(at 144.78 107.95 0)
 			(effects
@@
 			)
 		)
-		(property "MPN" "GRM32ER72A225KA35"
+		(property "MPN" "GRM32ER72A225KA35L"
 			(at 262.89 107.95 0)
 			(effects
@@
 			)
 		)
-		(property "MPN" "GRM32ER72A225KA35"
+		(property "MPN" "GRM32ER72A225KA35L"
 			(at 269.24 107.95 0)
 			(effects
@@
 			)
 		)
-		(property "MPN" "GRM32ER72A225KA35"
+		(property "MPN" "GRM32ER72A225KA35L"
 			(at 281.94 107.95 0)
 			(effects
@@
 			)
 		)
-		(property "MPN" "GRM32ER72A225KA35"
+		(property "MPN" "GRM32ER72A225KA35L"
 			(at 256.54 107.95 0)
 			(effects
@@
 			)
 		)
-		(property "MPN" "GRM32ER72A225KA35"
+		(property "MPN" "GRM32ER72A225KA35L"
 			(at 294.64 107.95 0)
 			(effects
@@
 			)
 		)
-		(property "MPN" "GRM32ER72A225KA35"
+		(property "MPN" "GRM32ER72A225KA35L"
 			(at 157.48 107.95 0)
 			(effects
@@
 			)
 		)
-		(property "MPN" "GRM32ER72A225KA35"
+		(property "MPN" "GRM32ER72A225KA35L"
 			(at 275.59 107.95 0)
 			(effects
@@
 			)
 		)
-		(property "MPN" "GRM32ER72A225KA35"
+		(property "MPN" "GRM32ER72A225KA35L"
 			(at 288.29 107.95 0)
 			(effects
@@
 			)
 		)
-		(property "MPN" "GRM32ER72A225KA35"
+		(property "MPN" "GRM32ER72A225KA35L"
 			(at 300.99 107.95 0)
 			(effects
@@
 			)
 		)
-		(property "MPN" "GRM32ER72A225KA35"
+		(property "MPN" "GRM32ER72A225KA35L"
 			(at 138.43 107.95 0)
 			(effects
@@
 			)
 		)
-		(property "MPN" "GRM32ER72A225KA35"
+		(property "MPN" "GRM32ER72A225KA35L"
 			(at 163.83 107.95 0)
 			(effects

Commit message: Add capacitor labels
Other:
- note added: "2.2uF 100V X7R"
Changed lines of the file:
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@@
+		)
+	)
+	(text "2.2uF 100V X7R"
+		(exclude_from_sim no)
+		(at 279.4 102.108 0)
+		(effects
+			(font
+				(size 1.27 1.27)
+			)
+		)
+	)
+	(text "2.2uF 100V X7R"
+		(exclude_from_sim no)
+		(at 151.13 102.108 0)
+		(effects
+			(font
+				(size 1.27 1.27)
+			)
 		)
 	)

Commit message: prune bogus symbol fields
Parts:
- U11: Availability In Stock -> (none); Check_prices https://www.snapeda.com/parts/PI3740-00-LGIZ/Vicor+Corporat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 -> (none); Description_1 Buck-Boost Switching Regulator IC Positive Adjustable (Fixe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 -> (none); MANUFACTURER VICOR -> (none); MF Vicor Corporation -> (none); MP PI3740-00-LGIZ -> (none); PARTREV 1.9 -> (none); Package BLGA-108 Vicor -> (none); Price None -> (none); STANDARD Manufacturer Recommendation -> (none); SnapEDA_Link https://www.snapeda.com/parts/PI3740-00-LGIZ/Vicor+Corporat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 -> (none)
Changed lines of the file:
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@@
-			)
-		)
-		(property "MF" "Vicor Corporation"
-			(at 214.63 129.54 0)
-			(effects
-				(font
-					(size 1.27 1.27)
-				)
-				(justify bottom)
-				(hide yes)
-			)
-		)
-		(property "Description_1" "\n                        \n                            Buck-Boost Switching Regulator IC Positive Adjustable (Fixed) 10V (12V) 1 Output 7.42A 108-BLGA Module\n                        \n"
-			(at 214.63 129.54 0)
-			(effects
-				(font
-					(size 1.27 1.27)
-				)
-				(justify bottom)
-				(hide yes)
-			)
-		)
-		(property "Package" "BLGA-108 Vicor"
-			(at 214.63 129.54 0)
-			(effects
-				(font
-					(size 1.27 1.27)
-				)
-				(justify bottom)
-				(hide yes)
-			)
-		)
-		(property "Price" "None"
-			(at 214.63 129.54 0)
-			(effects
-				(font
-					(size 1.27 1.27)
-				)
-				(justify bottom)
-				(hide yes)
-			)
-		)
-		(property "Check_prices" "https://www.snapeda.com/parts/PI3740-00-LGIZ/Vicor+Corporation/view-part/?ref=eda"
-			(at 214.63 129.54 0)
-			(effects
-				(font
-					(size 1.27 1.27)
-				)
-				(justify bottom)
-				(hide yes)
-			)
-		)
-		(property "STANDARD" "Manufacturer Recommendation"
-			(at 214.63 129.54 0)
-			(effects
-				(font
-					(size 1.27 1.27)
-				)
-				(justify bottom)
-				(hide yes)
-			)
-		)
-		(property "PARTREV" "1.9"
-			(at 214.63 129.54 0)
-			(effects
-				(font
-					(size 1.27 1.27)
-				)
-				(justify bottom)
-				(hide yes)
-			)
-		)
-		(property "SnapEDA_Link" "https://www.snapeda.com/parts/PI3740-00-LGIZ/Vicor+Corporation/view-part/?ref=snap"
-			(at 214.63 129.54 0)
-			(effects
-				(font
-					(size 1.27 1.27)
-				)
-				(justify bottom)
-				(hide yes)
-			)
-		)
-		(property "MP" "PI3740-00-LGIZ"
-			(at 214.63 129.54 0)
-			(effects
-				(font
-					(size 1.27 1.27)
-				)
-				(justify bottom)
-				(hide yes)
-			)
-		)
-		(property "Availability" "In Stock"
-			(at 214.63 129.54 0)
-			(effects
-				(font
-					(size 1.27 1.27)
-				)
-				(justify bottom)
-				(hide yes)
-			)
-		)
-		(property "MANUFACTURER" "VICOR"
-			(at 214.63 129.54 0)
-			(effects
-				(font
-					(size 1.27 1.27)
-				)
-				(justify bottom)
-				(hide yes)
 			)
 		)

Commit message: re-add all TPs but TP12 to BOM
Parts:
- TP10, TP11, TP8, TP9: now in the parts list
Changed lines of the file:
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@@
 		(unit 1)
 		(exclude_from_sim no)
-		(in_bom no)
+		(in_bom yes)
 		(on_board yes)
 		(dnp no)
@@
 		(unit 1)
 		(exclude_from_sim no)
-		(in_bom no)
+		(in_bom yes)
 		(on_board yes)
 		(dnp no)
@@
 		(unit 1)
 		(exclude_from_sim no)
-		(in_bom no)
+		(in_bom yes)
 		(on_board yes)
 		(dnp no)
@@
 		(unit 1)
 		(exclude_from_sim no)
-		(in_bom no)
-		(on_board yes)
-		(dnp no)
+		(in_bom yes)
+		(on_board yes)
+		(dnp no)

Commit message: connect inductor mounting pin to large ground area
Connections:
- net GND: now also L1.3 (MNT)
Changed lines of the file:
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@@
 	(wire
 		(pts
-			(xy 198.12 92.71) (xy 212.09 92.71)
+			(xy 198.12 85.09) (xy 209.55 85.09)
 		)
 		(stroke
@@
 	(wire
 		(pts
-			(xy 231.14 92.71) (xy 231.14 101.6)
+			(xy 231.14 85.09) (xy 231.14 101.6)
 		)
 		(stroke
@@
 	(wire
 		(pts
+			(xy 209.55 87.63) (xy 208.28 87.63)
+		)
+		(stroke
+			(width 0)
+			(type default)
+		)
+	)
+	(wire
+		(pts
 			(xy 236.22 139.7) (xy 236.22 142.24)
 		)
@@
 	(wire
 		(pts
+			(xy 208.28 87.63) (xy 208.28 88.9)
+		)
+		(stroke
+			(width 0)
+			(type default)
+		)
+	)
+	(wire
+		(pts
 			(xy 275.59 104.14) (xy 281.94 104.14)
 		)
@@
 	(wire
 		(pts
-			(xy 198.12 101.6) (xy 198.12 92.71)
+			(xy 198.12 101.6) (xy 198.12 85.09)
 		)
 		(stroke
@@
 	(wire
 		(pts
-			(xy 217.17 92.71) (xy 231.14 92.71)
+			(xy 219.71 85.09) (xy 231.14 85.09)
 		)
 		(stroke
@@
 	(symbol
 		(lib_id "Device:L_Small")
-		(at 214.63 92.71 90)
+		(at 214.63 83.82 90)
 		(unit 1)
 		(exclude_from_sim no)
@@
 		(fields_autoplaced yes)
 		(property "Reference" "L1"
-			(at 214.63 87.63 90)
+			(at 214.63 78.74 90)
 			(effects
 				(font
@@
 		)
 		(property "Value" "PA5119.421NLT"
-			(at 214.63 90.17 90)
+			(at 214.63 81.28 90)
 			(effects
 				(font
@@
 		)
 		(property "Footprint" "footprints:SMT_119.421NLT_PUL"
-			(at 214.63 92.71 0)
+			(at 214.63 83.82 0)
 			(effects
 				(font
@@
 		)
 		(property "Datasheet" "~"
-			(at 214.63 92.71 0)
+			(at 214.63 85.09 0)
 			(effects
 				(font
@@
 		)
 		(property "Description" "Inductor, small symbol"
-			(at 214.63 92.71 0)
+			(at 214.63 83.82 0)
 			(effects
 				(font
@@
 		)
 		(property "MPN" "PA5119.421NLT"
-			(at 214.63 92.71 0)
+			(at 214.63 83.82 0)
 			(effects
 				(font
@@
 					(unit 1)
 				)
+			)
+		)
+	)
+	(symbol
+		(lib_id "power:GND")
+		(at 208.28 88.9 0)
+		(mirror y)
+		(unit 1)
+		(exclude_from_sim no)
+		(in_bom yes)
+		(on_board yes)
+		(dnp no)
+		(property "Reference" "#PWR091"
+			(at 208.28 95.25 0)
+			(effects
+				(font
+					(size 1.27 1.27)
+				)
+				(hide yes)
+			)
+		)
+		(property "Value" "GND"
+			(at 208.28 93.98 0)
+			(effects
+				(font
+					(size 1.27 1.27)
+				)
+				(hide yes)
+			)
+		)
+		(property "Footprint" ""
+			(at 208.28 88.9 0)
+			(effects
+				(font
+					(size 1.27 1.27)
+				)
+				(hide yes)
+			)
+		)
+		(property "Datasheet" ""
+			(at 208.28 88.9 0)
+			(effects
+				(font
+					(size 1.27 1.27)
+				)
+				(hide yes)
+			)
+		)
+		(property "Description" ""
+			(at 208.28 88.9 0)
+			(effects
+				(font
+					(size 1.27 1.27)
+				)
+				(hide yes)
+			)
+		)
+		(pin "1"
+		)
+		(instances
+			(project "roadster-charger"
+				(path "/57ecac41-cd8a-4182-a81e-fed3e381aedd/64ca4e4e-11ba-4e5c-8f8e-2432a1d47dd0"
+					(reference "#PWR091")
+					(unit 1)
+				)
